File: placa de interface clp.kicad_pcb (KiCad board)
At the start: 2 copper layers, 41 parts, among them J1 Screw_Terminal_01x02, J10 Screw_Terminal_01x02, J11 Screw_Terminal_01x02, J12 Screw_Terminal_01x02, J2 Screw_Terminal_01x02, J3 Screw_Terminal_01x02, J4 Screw_Terminal_01x02, J5 Screw_Terminal_01x02, J6 Screw_Terminal_01x02, J7 Screw_Terminal_01x02, J8 Screw_Terminal_01x02, J9 Screw_Terminal_01x02, SW1 SW_SPDT_312, U1 EL817, U4 EL817, U5 EL817, U6 EL817, U7 EL817, U8 EL817, U9 EL817

Commit message: ATT 4
Parts:
- removed J12, J2, J3: Screw_Terminal_01x02, TerminalBlock_Phoenix:TerminalBlock_Phoenix_MKDS-1,5-2_1x02_P5.00mm_Horizontal
- added H1: MountingHole_Pad, MountingHole:MountingHole_2.5mm_Pad, F.Cu at (97.0, 106.0)
- added H2: MountingHole_Pad, MountingHole:MountingHole_2.5mm_Pad, F.Cu at (97.0, 115.0)
- added H3: MountingHole_Pad, MountingHole:MountingHole_2.5mm_Pad, F.Cu at (137.0, 130.0)
- added H4: MountingHole_Pad, MountingHole:MountingHole_2.5mm_Pad, F.Cu at (137.0, 139.0)
- moved J10 131.0 mm to (64.0, 143.3)
- moved R13 92.7 mm to (193.5, 80.6), turned to -90 degrees
- moved J7 87.1 mm to (68.8, 76.7), turned to 180 degrees
- moved J1 86.8 mm to (56.7, 107.5), turned to -90 degrees
- moved J4 86.3 mm to (113.5, 143.0)
- moved J5 85.8 mm to (92.0, 143.0)
- moved SW1 85.5 mm to (77.0, 110.0), turned to 90 degrees
- moved D6 78.5 mm to (65.0, 134.0), turned to 90 degrees
- moved R3 75.7 mm to (84.5, 138.7), turned to 90 degrees
- moved R14 71.8 mm to (173.5, 90.8), turned to 90 degrees
- moved U9 67.4 mm to (185.1, 94.7), turned to 180 degrees
- moved U4 65.1 mm to (92.5, 124.4)
- moved R11 63.0 mm to (56.5, 139.0), turned to 90 degrees
- moved U1 62.7 mm to (68.3, 96.3), turned to 180 degrees
- moved U8 62.5 mm to (65.0, 124.7)
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Routing:
- net Earth: track 0.00 -> 345.9 mm
- net +24V: track 0.00 -> 156.6 mm
- net +5V: track 0.00 -> 80.5 mm
- net /IN+: track 0.00 -> 22.8 mm
- net Net-(R11-Pad2): track 0.00 -> 11.4 mm
- net Net-(R13-Pad2): track 0.00 -> 11.4 mm
- net /ESP_SIG_7: track 0.00 -> 11.2 mm
- net Net-(R5-Pad2): track 0.00 -> 10.9 mm
- net /ESP_SIG_6: track 0.00 -> 10.7 mm
- net /CLP_SIG_3: track 0.00 -> 10.7 mm
- net /CLP_SIG_1: track 0.00 -> 10.6 mm
- net /CLP_SIG_2: track 0.00 -> 10.6 mm
- net Net-(R3-Pad2): track 0.00 -> 10.4 mm
- net /CLP_SIG_5: track 0.00 -> 10.4 mm
- net /ESP_SIG_5: track 0.00 -> 10.4 mm
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Other:
- board outline added: 150 x 80.2 mm
- board text added: "24V"
- board text added: "5V"
- board text added: "GND"
- board text added: "IN+"
- board text added: "IN-"
- board text added: "L298N"
- board text added: "LM2596"
