File: PLACA/placa de interface clp.kicad_pcb (KiCad board)
At the start: 2 copper layers, 150 x 80.2 mm, 42 parts, among them J1 Screw_Terminal_01x02, J10 Screw_Terminal_01x02, J11 Screw_Terminal_01x02, J4 Screw_Terminal_01x02, J5 Screw_Terminal_01x02, J6 Screw_Terminal_01x02, J7 Screw_Terminal_01x02, J8 Screw_Terminal_01x02, J9 Screw_Terminal_01x02, SW1 SW_SPDT_312, U1 EL817, U4 EL817, U5 EL817, U6 EL817, U7 EL817, U8 EL817, U9 EL817

Commit message: ATT 8
Routing:
- net Net-(R9-Pad2): track 9.16 -> 10.0 mm
